Commit message: URDF

File: src/diffdrive_arduino/description/urdf/diffbot_description.urdf.xacro (robot description, xacro)
@@ -2,160 +2,112 @@
 <robot xmlns:xacro="http://www.ros.org/wiki/xacro">
   <xacro:macro name="diffbot" params="prefix">
-  <!-- Constants for robot dimensions -->
-  <xacro:property name="PI" value="3.1415926535897931"/>
-  <xacro:property name="base_mass" value="0.3" /> <!-- arbitrary value for base mass -->
-  <xacro:property name="base_width" value="0.1" />
-  <xacro:property name="base_length" value="0.1" />
-  <xacro:property name="base_height" value="0.05" />
-  <xacro:property name="wheel_mass" value="0.3" /> <!-- arbitrary value for wheel mass -->
-  <xacro:property name="wheel_len" value="0.020" />
-  <xacro:property name="wheel_radius" value="0.015" />
-  <xacro:property name="caster_wheel_mass" value="0.1" /> <!-- arbitrary value for caster wheel mass -->
-  <xacro:property name="caster_wheel_radius" value="0.015" />
-  <xacro:property name="z_offset" value="-${base_height/2}" /> <!-- Space btw top of beam and the each joint -->
-  <!-- Base Link -->
-  <link name="${prefix}base_link">
-    <collision>
-      <origin xyz="0 0 0" rpy="0 0 0"/>
-      <geometry>
-        <box size="${base_width} ${base_length} ${base_height}"/>
-      </geometry>
-    </collision>
-    <visual>
-      <origin xyz="0 0 ${base_height/2}" rpy="0 0 0"/>
-      <geometry>
-        <box size="${base_width} ${base_length} ${base_height}"/>
-      </geometry>
-      <material name="orange"/>
-    </visual>
-    <inertial>
-      <origin xyz="0 0 0" rpy="0 0 0"/>
-      <mass value="${base_mass}"/>
-      <inertia
-        ixx="${base_mass / 12.0 * (base_length*base_length + base_height*base_height)}" ixy="0.0" ixz="0.0"
-        iyy="${base_mass / 12.0 * (base_height*base_height + base_width*base_width)}" iyz="0.0"
-        izz="${base_mass / 12.0 * (base_width*base_width + base_length*base_length)}"/>
+    <!-- Define robot constants -->
+    <xacro:property name="base_width" value="0.119"/>
+    <xacro:property name="base_length" value="0.152"/>
+    <xacro:property name="base_height" value="0.083"/>
+    <xacro:property name="wheel_radius" value="0.0325"/>
+    <xacro:property name="wheel_width" value="0.025"/>
+    <xacro:property name="wheel_ygap" value="0.0155"/>
+    <xacro:property name="wheel_zoff" value="0.026"/>
+    <xacro:property name="wheel_xoff" value="0.02"/>
+    <xacro:property name="caster_xoff" value="0.061"/>
+    <!-- Define intertial property macros  -->
+    <xacro:macro name="box_inertia" params="m w h d">
+      <inertial>
+        <origin xyz="0 0 0" rpy="${pi/2} 0 ${pi/2}"/>
+        <mass value="${m}"/>
+        <inertia ixx="${(m/12) * (h*h + d*d)}" ixy="0.0" ixz="0.0" iyy="${(m/12) * (w*w + d*d)}" iyz="0.0" izz="${(m/12) * (w*w + h*h)}"/>
       </inertial>
-    </link>
-    <joint name="${prefix}left_wheel_joint" type="continuous">
-      <parent link="${prefix}base_link"/>
-      <child link="${prefix}left_wheel"/>
-      <origin xyz="0 -${base_width/2} ${z_offset}" rpy="0 0 0"/>
-      <axis xyz="0 1 0"/>
-      <dynamics damping="0.2"/>
-    </joint>
-    <!-- left wheel Link -->
-    <link name="${prefix}left_wheel">
+    </xacro:macro>
+    <xacro:macro name="cylinder_inertia" params="m r h">
+      <inertial>
+        <origin xyz="0 0 0" rpy="${pi/2} 0 0" />
+        <mass value="${m}"/>
+        <inertia ixx="${(m/12) * (3*r*r + h*h)}" ixy = "0" ixz = "0" iyy="${(m/12) * (3*r*r + h*h)}" iyz = "0" izz="${(m/2) * (r*r)}"/>
+      </inertial>
+    </xacro:macro>
+    <xacro:macro name="sphere_inertia" params="m r">
+      <inertial>
+        <mass value="${m}"/>
+        <inertia ixx="${(2/5) * m * (r*r)}" ixy="0.0" ixz="0.0" iyy="${(2/5) * m * (r*r)}" iyz="0.0" izz="${(2/5) * m * (r*r)}"/>
+      </inertial>
+    </xacro:macro>
+    <!-- Robot Base -->
+    <link name="${prefix}base_link">
+      <visual>
+        <origin xyz="0 0 ${(wheel_zoff+wheel_radius)}" rpy="0 0 0"/>
+        <geometry>
+          <box size="${base_length} ${base_width} ${base_height}"/>
+        </geometry>
+        <material name="Cyan">
+          <color rgba="0 1.0 1.0 1.0"/>
+        </material>
+      </visual>
       <collision>
-        <origin xyz="0 0 0" rpy="${PI/2} 0 0"/>
         <geometry>
-          <cylinder length="${wheel_len}" radius="${wheel_radius}"/>
+          <box size="${base_length} ${base_width} ${base_height}"/>
         </geometry>
       </collision>
+      <xacro:box_inertia m="15" w="${base_width}" d="${base_length}" h="${base_height}"/>
+    </link>
+    <!-- Robot Footprint -->
+    <link name="base_footprint"/>
+    <joint name="base_joint" type="fixed">
+      <parent link="${prefix}base_link"/>
+      <child link="base_footprint"/>
+      <origin xyz="0.0 0.0 ${(wheel_zoff+wheel_radius)}" rpy="0 0 0"/>
+    </joint>
+    <!-- Wheels -->
+    <xacro:macro name="wheel" params="wheel_name x_reflect y_reflect">
+      <link name="${wheel_name}">
+        <visual>
+          <origin xyz="0 0 0" rpy="${pi/2} 0 0"/>
+          <geometry>
+              <cylinder radius="${wheel_radius}" length="${wheel_width}"/>
+          </geometry>
+          <material name="Gray">
+            <color rgba="0.5 0.5 0.5 1.0"/>
+          </material>
+        </visual>
+        <collision>
+          <origin xyz="0 0 0" rpy="${pi/2} 0 0"/>
+          <geometry>
+            <cylinder radius="${wheel_radius}" length="${wheel_width}"/>
+          </geometry>
+        </collision>
+        <xacro:cylinder_inertia m="0.5" r="${wheel_radius}" h="${wheel_width}"/>
+      </link>
+      <joint name="${wheel_name}_joint" type="continuous">
+        <parent link="${prefix}base_footprint"/>
+        <child link="${wheel_name}"/>
+        <origin xyz="${x_reflect*wheel_xoff} ${y_reflect*(base_width/2+wheel_ygap)} ${-wheel_zoff}" rpy="0 0 0"/>
+        <axis xyz="0 1 0"/>
+      </joint>
+    </xacro:macro>
+    <xacro:wheel wheel_name="${prefix}left_wheel" x_reflect="1" y_reflect="1" />
+    <xacro:wheel wheel_name="${prefix}right_wheel" x_reflect="1" y_reflect="-1" />
+    <!-- Caster Wheel -->
+    <link name="${prefix}caster_rear_wheel">
       <visual>
-        <origin xyz="0 0 0" rpy="${PI/2} 0 0"/>
         <geometry>
-          <cylinder length="${wheel_len}" radius="${wheel_radius}"/>
+          <sphere radius="${((wheel_radius)+wheel_zoff-(base_height/2))}"/>
         </geometry>
-        <material name="black"/>
+        <material name="Cyan">
+          <color rgba="0 1.0 1.0 1.0"/>
+        </material>
       </visual>
-      <inertial>
-        <origin xyz="0 0 0" rpy="${PI/2} 0 0"/>
-        <mass value="${wheel_mass}"/>
-        <inertia
-          ixx="${wheel_mass / 12.0 * (3*wheel_radius + wheel_len*wheel_len)}" ixy="0.0" ixz="0.0"
-          iyy="${wheel_mass / 12.0 * wheel_radius*wheel_radius}" iyz="0.0"
-          izz="${wheel_mass / 12.0 * wheel_radius*wheel_radius}"/>
-        </inertial>
-      </link>
-    <joint name="${prefix}right_wheel_joint" type="continuous">
-      <parent link="${prefix}base_link"/>
-      <child link="${prefix}right_wheel"/>
-      <origin xyz="0 ${base_width/2} ${z_offset}" rpy="0 0 0"/>
-      <axis xyz="0 1 0"/>
-      <dynamics damping="0.2"/>
-    </joint>
-    <!-- right wheel Link -->
-    <link name="${prefix}right_wheel">
-      <collision>
-        <origin xyz="0 0 0" rpy="${PI/2} 0 0"/>
-        <geometry>
-          <cylinder length="${wheel_len}" radius="${wheel_radius}"/>
-        </geometry>
-      </collision>
-      <visual>
-        <origin xyz="0 0 0" rpy="${PI/2} 0 0"/>
-        <geometry>
-          <cylinder length="${wheel_len}" radius="${wheel_radius}"/>
-        </geometry>
-        <material name="black"/>
-      </visual>
-      <inertial>
-        <origin xyz="0 0 0" rpy="${PI/2} 0 0"/>
-        <mass value="${wheel_mass}"/>
-        <inertia
-          ixx="${wheel_mass / 12.0 * (3*wheel_radius + wheel_len*wheel_len)}" ixy="0.0" ixz="0.0"
-          iyy="${wheel_mass / 12.0 * wheel_radius*wheel_radius}" iyz="0.0"
-          izz="${wheel_mass / 12.0 * wheel_radius*wheel_radius}"/>
-        </inertial>
-      </link>
-    <joint name="${prefix}caster_frontal_wheel_joint" type="fixed">
-      <parent link="${prefix}base_link"/>
-      <child link="${prefix}caster_frontal_wheel"/>
-      <origin xyz="${base_width/2 - caster_wheel_radius} 0 ${z_offset}" rpy="0 0 0"/>
-    </joint>
-    <!-- caster frontal wheel Link -->
-    <link name="${prefix}caster_frontal_wheel">
       <collision>
         <origin xyz="0 0 0" rpy="0 0 0"/>
         <geometry>
-          <sphere radius="${caster_wheel_radius}"/>
+          <sphere radius="${((wheel_radius)+wheel_zoff-(base_height/2))}"/>
         </geometry>
       </collision>
-      <visual>
-        <origin xyz="0 0 0" rpy="0 0 0"/>
-        <geometry>
-          <sphere radius="${caster_wheel_radius}"/>
-        </geometry>
-        <material name="white"/>
-      </visual>
-      <inertial>
-        <origin xyz="0 0 0" rpy="0 0 0"/>
-        <mass value="${caster_wheel_mass}"/>
-        <inertia
-          ixx="${caster_wheel_mass * 0.4 * (caster_wheel_radius * caster_wheel_radius)}" ixy="0.0" ixz="0.0"
-          iyy="${caster_wheel_mass * 0.4 * (caster_wheel_radius * caster_wheel_radius)}" iyz="0.0"
-          izz="${caster_wheel_mass * 0.4 * (caster_wheel_radius * caster_wheel_radius)}"/>
-        </inertial>
-      </link>
+      <xacro:sphere_inertia m="0.5" r="${(wheel_radius+wheel_zoff-(base_height/2))}"/>
+    </link>
     <joint name="${prefix}caster_rear_wheel_joint" type="fixed">
-      <parent link="${prefix}base_link"/>
+      <parent link="${prefix}base_footprint"/>
       <child link="${prefix}caster_rear_wheel"/>
-      <origin xyz="${-base_width/2 + caster_wheel_radius} 0 ${z_offset}" rpy="0 0 0"/>
+      <origin xyz="${-caster_xoff} 0.0 ${-(base_height/2)}" rpy="0 0 0"/>
     </joint>
-    <!-- caster rear wheel Link -->
-    <link name="${prefix}caster_rear_wheel">
-      <collision>
-        <origin xyz="0 0 0" rpy="0 0 0"/>
-        <geometry>
-          <sphere radius="${caster_wheel_radius}"/>
-        </geometry>
-      </collision>
-      <visual>
-        <origin xyz="0 0 0" rpy="0 0 0"/>
-        <geometry>
-          <sphere radius="${caster_wheel_radius}"/>
-        </geometry>
-        <material name="white"/>
-      </visual>
-      <inertial>
-        <origin xyz="0 0 0" rpy="0 0 0"/>
-        <mass value="${caster_wheel_mass}"/>
-        <inertia
-          ixx="${caster_wheel_mass * 0.4 * (caster_wheel_radius * caster_wheel_radius)}" ixy="0.0" ixz="0.0"
-          iyy="${caster_wheel_mass * 0.4 * (caster_wheel_radius * caster_wheel_radius)}" iyz="0.0"
-          izz="${caster_wheel_mass * 0.4 * (caster_wheel_radius * caster_wheel_radius)}"/>
-        </inertial>
-      </link>
   </xacro:macro>
 </robot>

Commit message: attempt to add mesh STL

File: src/diffdrive_arduino/description/urdf/diffbot_description.urdf.xacro (robot description, xacro)
@@ -38,5 +38,5 @@
         <origin xyz="0 0 ${(wheel_zoff+wheel_radius)}" rpy="0 0 0"/>
         <geometry>
-          <box size="${base_length} ${base_width} ${base_height}"/>
+          <mesh filename="file://$(find diffdrive_arduino)/meshes/Penguin_Pi_Model.STL" scale="1.0 1.0 1.0"/>
         </geometry>
         <material name="Cyan">
@@ -46,5 +46,5 @@
       <collision>
         <geometry>
-          <box size="${base_length} ${base_width} ${base_height}"/>
+          <mesh filename="file://$(find diffdrive_arduino)/meshes/Penguin_Pi_Model.STL" scale="1.0 1.0 1.0"/>
         </geometry>
       </collision>

Commit message: use dae instead of stl

File: src/diffdrive_arduino/description/urdf/diffbot_description.urdf.xacro (robot description, xacro)
@@ -38,5 +38,5 @@
         <origin xyz="0 0 ${(wheel_zoff+wheel_radius)}" rpy="0 0 0"/>
         <geometry>
-          <mesh filename="file://$(find diffdrive_arduino)/meshes/Penguin_Pi_Model.STL" scale="1.0 1.0 1.0"/>
+          <mesh filename="file://$(find diffdrive_arduino)/meshes/Penguin_Pi_Model.dae" scale="1.0 1.0 1.0"/>
         </geometry>
         <material name="Cyan">
@@ -46,5 +46,5 @@
       <collision>
         <geometry>
-          <mesh filename="file://$(find diffdrive_arduino)/meshes/Penguin_Pi_Model.STL" scale="1.0 1.0 1.0"/>
+          <mesh filename="file://$(find diffdrive_arduino)/meshes/Penguin_Pi_Model.dae" scale="1.0 1.0 1.0"/>
         </geometry>
       </collision>

Commit message: dae file not working, I need to rotate it

File: src/diffdrive_arduino/description/urdf/diffbot_description.urdf.xacro (robot description, xacro)
@@ -38,5 +38,6 @@
         <origin xyz="0 0 ${(wheel_zoff+wheel_radius)}" rpy="0 0 0"/>
         <geometry>
-          <mesh filename="file://$(find diffdrive_arduino)/meshes/Penguin_Pi_Model.dae" scale="1.0 1.0 1.0"/>
+          <!-- <mesh filename="file://$(find diffdrive_arduino)/meshes/Penguin_Pi_Model.dae" scale="1.0 1.0 1.0"/> -->
+          <box size="${base_length} ${base_width} ${base_height}"/>
         </geometry>
         <material name="Cyan">
@@ -46,5 +47,6 @@
       <collision>
         <geometry>
-          <mesh filename="file://$(find diffdrive_arduino)/meshes/Penguin_Pi_Model.dae" scale="1.0 1.0 1.0"/>
+          <!-- <mesh filename="file://$(find diffdrive_arduino)/meshes/Penguin_Pi_Model.dae" scale="1.0 1.0 1.0"/> -->
+          <box size="${base_length} ${base_width} ${base_height}"/>
         </geometry>
       </collision>
