Commit message: fixed naming from diffdrive_arduino to diffdrive_penguinpi

File: src/diffdrive_penguinpi/description/ros2_control/diffbot.ros2_control.xacro (robot description, xacro)
@@ -4,5 +4,5 @@
     <ros2_control name="${name}" type="system">
       <hardware>
-        <plugin>diffdrive_arduino/DiffDriveArduinoHardware</plugin>
+        <plugin>diffdrive_penguinpi/DiffDrivePenguinPiHardware</plugin>
         <param name="left_wheel_name">left_wheel_joint</param>
           <param name="right_wheel_name">right_wheel_joint</param>

File: src/diffdrive_penguinpi/description/urdf/diffbot.urdf.xacro (robot description, xacro)
@@ -3,9 +3,9 @@
 <robot xmlns:xacro="http://www.ros.org/wiki/xacro" name="diffdrive_robot">
   <xacro:arg name="prefix" default="" />
-  <xacro:include filename="$(find diffdrive_arduino)/urdf/diffbot_description.urdf.xacro" />
+  <xacro:include filename="$(find diffdrive_penguinpi)/urdf/diffbot_description.urdf.xacro" />
   <!-- Import Rviz colors -->
-  <xacro:include filename="$(find diffdrive_arduino)/urdf/diffbot.materials.xacro" />
+  <xacro:include filename="$(find diffdrive_penguinpi)/urdf/diffbot.materials.xacro" />
   <!-- Import diffbot ros2_control description -->
-  <xacro:include filename="$(find diffdrive_arduino)/ros2_control/diffbot.ros2_control.xacro" />
+  <xacro:include filename="$(find diffdrive_penguinpi)/ros2_control/diffbot.ros2_control.xacro" />
   <xacro:diffbot prefix="$(arg prefix)" />
   <xacro:diffbot_ros2_control

File: src/diffdrive_penguinpi/description/urdf/diffbot_description.urdf.xacro (robot description, xacro)
@@ -38,5 +38,5 @@
         <origin xyz="0 0 ${(wheel_zoff+wheel_radius)}" rpy="0 0 0"/>
         <geometry>
-          <!-- <mesh filename="file://$(find diffdrive_arduino)/meshes/Penguin_Pi_Model.dae" scale="1.0 1.0 1.0"/> -->
+          <!-- <mesh filename="file://$(find diffdrive_penguinpi)/meshes/Penguin_Pi_Model.dae" scale="1.0 1.0 1.0"/> -->
           <box size="${base_length} ${base_width} ${base_height}"/>
         </geometry>
@@ -47,5 +47,5 @@
       <collision>
         <geometry>
-          <!-- <mesh filename="file://$(find diffdrive_arduino)/meshes/Penguin_Pi_Model.dae" scale="1.0 1.0 1.0"/> -->
+          <!-- <mesh filename="file://$(find diffdrive_penguinpi)/meshes/Penguin_Pi_Model.dae" scale="1.0 1.0 1.0"/> -->
           <box size="${base_length} ${base_width} ${base_height}"/>
         </geometry>
